Commit message: Typo: torso.std to torso.stl

File: robots/hsrb4s.urdf (robot description, URDF)
Before this commit: robot hsrb, 45 links, 44 joints
Links:
- link torso_lift_link: geometry collision mesh filename=package://hsr_meshes/meshes/torso_v0/torso.stl; visual mesh filename=package://hsr_meshes/meshes/torso_v0/torso_light.dae
